File: KiCad/fancontroller/fancontroller.kicad_pcb (KiCad board)
At the start: 2 copper layers, 25.7 x 36.8 mm, 0 parts

Commit message: feat: place recovered SMD footprints and record draft assembly positions
Parts:
- added C1: 560pF, Capacitor_SMD:C_1206_3216Metric, F.Cu at (81.3, 160.9)
- added C2: 100nF, Capacitor_SMD:C_0603_1608Metric, F.Cu at (95.0, 155.4)
- added C3: 100nF, Capacitor_SMD:C_0603_1608Metric, F.Cu at (95.0, 164.6)
- added C4: 100pF, Capacitor_SMD:C_1206_3216Metric, F.Cu at (96.5, 172.4)
- added C5: 47uF 10V, Capacitor_SMD:CP_Elec_6.3x5.8, F.Cu at (84.3, 147.6)
- added IC1: NE555DR, Package_SO:SOIC-8_3.9x4.9mm_P1.27mm, F.Cu at (95.9, 150.5)
- added IC2: LM311DR, Package_SO:SOIC-8_3.9x4.9mm_P1.27mm, F.Cu at (90.2, 158.5)
- added IC3: NE555DR, Package_SO:SOIC-8_3.9x4.9mm_P1.27mm, F.Cu at (90.2, 167.6)
- added R1: 10k, Resistor_SMD:R_1206_3216Metric, F.Cu at (81.3, 154.4)
- added R2: 47k, Resistor_SMD:R_1206_3216Metric, F.Cu at (81.3, 157.5)
- added R3: 9.1k, Resistor_SMD:R_1206_3216Metric, F.Cu at (81.3, 164.5)
- added R4: 9.1k, Resistor_SMD:R_1206_3216Metric, F.Cu at (81.3, 167.5)
- added R5: 1k, Resistor_SMD:R_1206_3216Metric, F.Cu at (90.3, 162.6)
- added REG1: TS2938CS50, Package_SO:SOIC-8_3.9x4.9mm_P1.27mm, F.Cu at (89.6, 143.4)
Routing:
- net 0: track 747.3 -> 0.00 mm
- net (no net): track 0.00 -> 747.3 mm
