File: KiCad/fancontroller/fancontroller.kicad_pcb (KiCad board)
At the start: 2 copper layers, 25.7 x 36.8 mm, 21 parts, among them IC1 NE555DR, IC2 LM311DR, IC3 NE555DR, J1 Fan 4-pin, J2 Power input, P1 10k

Commit message: feat: clear native ERC and DRC and export revised 12 V assembly candidate
Parts:
- added C6: 100nF, Recovered2018:C_0603_1608Metric_Pad1.05x0.95mm_HandSolder, F.Cu at (96.0, 141.4)
Routing:
- net +12V: track 30.2 -> 33.6 mm
- net DUTY_REF: track 28.5 -> 27.2 mm
- net GND: track 47.4 -> 48.3 mm, vias 15 -> 16
Other:
- board text added: "+"
- board text added: "-"
- board text added: "1 GND"
- board text added: "2 +12"
- board text added: "3 NC"
- board text added: "4 PWM"
- board text added: "C2"
- board text added: "C3"
- board text added: "C5"
- board text added: "IC3"
- board text added: "J1"
- board text added: "J2"
- board text added: "PWM FAN 12V"
- board text added: "R2"
- board text added: "R4"
- board text added: "R5"
